File: RC-1.sch (KiCad schematic (older format))
At the start: 46 parts, among them P1 PCIe_M.2_B-Key, U1 STM32F401CEUx, U2 ADF7021, Y1 8MHz

Commit message: Add old changes from 3 Aug 2021
Parts:
- added AE1: Ceramic Antenna, symbol Device:Antenna_Dipole
- added C2, C3: 100n, Capacitor_SMD:C_0402_1005Metric, symbol Device:C
- added J1: U.FL, Connector_Coaxial:U.FL_Hirose_U.FL-R-SMT-1_Vertical, symbol Connector:Conn_Coaxial
- C1, C10, C12, C14, C15, C17, C18, C20, C22, C23, C25, C26, C27, C28, C4, C5, C6, C7, C9: renamed from C?; footprint (none) -> Capacitor_SMD:C_0402_1005Metric
- L1, L2, L3: renamed from L?; footprint (none) -> Inductor_SMD:L_0402_1005Metric
- R1, R10, R11, R2, R3, R4, R5, R7, R8, R9: renamed from R?; footprint (none) -> Resistor_SMD:R_0402_1005Metric
- gave numbers to parts that had none: 4
- renumbered C4 to C11, C5 to C13, C1 to C16, C2 to C19, C3 to C8, R1 to R6
Connections:
- net I2S_IN_SCK is gone; now on net SPI2_MISO: P1.46 (GPIO_3_(I/O)_(0/3.3V))
- net I2S_IN_WS is gone; now on net SPI2_MOSI: P1.48 (GPIO_4_(I/O)_(0/3.3V))
- net SPI_CS is gone; now on net SPI1_CS: P1.65 (ANTCTL3_(I)_(0/1.8V))
- net SPI_MISO is gone; now on net SPI1_MISO: P1.61 (ANTCTL1_(I)_(0/1.8V))
- net SPI_MOSI is gone; now on net SPI1_MOSI: P1.63 (ANTCTL2_(I)_(0/1.8V))
- net SPI_SCLK is gone; now on net SPI1_SCLK: P1.59 (ANTCTL0_(I)_(0/1.8V))
- net CLKOUT: no longer U1.46 (PB9)
- net DATAIN: no longer U1.21 (PB10)
- net DATAOUT: no longer U1.25 (PB12)
- net GND: now also J1.2 (Ext)
- net I2C_SCL: now also U1.42 (PB6)
- net I2C_SDA: now also U1.43 (PB7)
- net RF: now also C2.2, C3.2
- net SCLK: no longer U1.41 (PB5)
- net SDATA: no longer U1.42 (PB6)
- net SLE: no longer U1.45 (PB8)
- net SREAD: no longer U1.43 (PB7)
- net SPI1_CS: now reaches U1.14 (PA4)
- net SPI1_SCLK: now reaches U1.15 (PA5)
- net SPI1_MISO: now reaches U1.16 (PA6)
- net SPI1_MOSI: now reaches U1.17 (PA7)
- net SPI2_SCLK: now reaches U1.26 (PB13)
- net SPI2_SCLK: now also P1.44 (GPIO_2_(I/O)_(0/3.3V))
- net SPI2_MISO: now reaches U1.27 (PB14)
- net SPI2_MOSI: now reaches U1.28 (PB15)
- net PTT: now reaches P1.26 (GPIO_10_(I/O)_(0/1.8V))
- net AUDIO_IN: now reaches P1.52 (CLKREQ#_(I/O)_(0/3.3V))
- net AUDIO_OUT: now reaches P1.54 (PEWAKE#_(I/O)_(0/3.3V))
- net I2S_IN_SD renamed SPI2_CS
- net SPI2_CS: now also U1.25 (PB12)
- net I2S_OUT_SCK renamed I2S_SCK
- net I2S_OUT_SD renamed I2S_SD
- net I2S_OUT_WS renamed I2S_WS
- new net: C2.1, J1.1 (In)
- new net: AE1.2, C3.1
- no-connect marks 40 -> 41
